File: demos/custom_pads_test/custom_pads_test.kicad_pcb (KiCad board)
At the start: 2 copper layers, 118 x 90 mm, 5 parts, among them SW1 R

Commit message: feat: update kicad to 9.0.0+dfsg-1
Signed-off-by: lhdjply <lhdjply@126.com>
Parts:
- AE1, AE2: footprint Connect:1pin -> custom_pads_test:1pin
- R2: footprint Diodes_SMD:DO-214AB -> custom_pads_test:DO-214AB
- SW1: footprint Discret:C2 -> custom_pads_test:C2
- U***: footprint Dip_sockets:DIP-14__300_ELL -> custom_pads_test:DIP-14__300_ELL
