File: demos/flat_hierarchy/pic_programmer.kicad_sch (KiCad schematic)
At the start: 56 parts, among them J1 DB9-FEMAL, P1 CONN_2, Q1 BC237, Q2 BC307, Q3 BC307, U2 74HC125, U3 7805, U4 LT1373

Commit message: feat: update kicad to 9.0.0+dfsg-1
Signed-off-by: lhdjply <lhdjply@126.com>
Parts:
- C1, C2, C3: symbol flat_hierarchy_schlib:CP -> flat_hierarchy:CP
- C4, C5, C9: symbol flat_hierarchy_schlib:C -> flat_hierarchy:C
- D1: symbol flat_hierarchy_schlib:D -> flat_hierarchy:D
- D10, D11, D2, D3, D4, D5, D6, D7: symbol flat_hierarchy_schlib:D_Schottky -> flat_hierarchy:D_Schottky
- D12, D8, D9: symbol flat_hierarchy_schlib:LED -> flat_hierarchy:LED
- HOLE1, HOLE2, HOLE3, HOLE4, HOLE5, HOLE6: symbol flat_hierarchy_schlib:CONN_1 -> flat_hierarchy:CONN_1
- J1: symbol flat_hierarchy_schlib:DB9 -> flat_hierarchy:DB9
- JP1: symbol flat_hierarchy_schlib:JUMPER -> flat_hierarchy:JUMPER
- L1: symbol flat_hierarchy_schlib:INDUCTOR -> flat_hierarchy:INDUCTOR
- P1: symbol flat_hierarchy_schlib:CONN_2 -> flat_hierarchy:CONN_2
- Q1: symbol flat_hierarchy_schlib:BC237 -> flat_hierarchy:BC237
- Q2, Q3: symbol flat_hierarchy_schlib:BC307 -> flat_hierarchy:BC307
- R1, R10, R11, R12, R13, R14, R15, R16, R17, R18, R19, R2, R20, R21, R3, R4, R5, R6, R7, R8, R9: symbol flat_hierarchy_schlib:R -> flat_hierarchy:R
- RV1: symbol flat_hierarchy_schlib:POT -> flat_hierarchy:POT
- U2: symbol flat_hierarchy_schlib:74LS125 -> flat_hierarchy:74LS125
- U3: symbol flat_hierarchy_schlib:7805 -> flat_hierarchy:7805
- U4: symbol flat_hierarchy_schlib:LT1373 -> flat_hierarchy:LT1373
