File: demos/flat_hierarchy/pic_sockets.kicad_sch (KiCad schematic)
At the start: 8 parts, among them P2 SUPP28, P3 SUPP40, U1 24Cxx, U5 PIC_18_PINS, U6 PIC_8_PINS

Commit message: feat: update kicad to 9.0.0+dfsg-1
Signed-off-by: lhdjply <lhdjply@126.com>
Parts:
- C6, C7, C8: symbol flat_hierarchy_schlib:C -> flat_hierarchy:C
- P2: symbol flat_hierarchy_schlib:SUPP28 -> flat_hierarchy:SUPP28
- P3: symbol flat_hierarchy_schlib:SUPP40 -> flat_hierarchy:SUPP40
- U1: symbol flat_hierarchy_schlib:24C16 -> flat_hierarchy:24C16
- U5: symbol flat_hierarchy_schlib:PIC16F54 -> flat_hierarchy:PIC16F54
- U6: symbol flat_hierarchy_schlib:PIC12C508A -> flat_hierarchy:PIC12C508A
Changed lines of the file:
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@@
 (kicad_sch
-	(version 20231120)
+	(version 20250114)
 	(generator "eeschema")
-	(generator_version "8.0")
+	(generator_version "9.0")
 	(paper "A4")
 	(title_block
@@
 	(label "DATA-RB7"
 		(at 229.87 101.6 0)
-		(fields_autoplaced yes)
 		(effects
 			(font
@@
 	(label "VCC_PIC"
 		(at 109.22 123.19 0)
-		(fields_autoplaced yes)
 		(effects
 			(font
@@
 	(label "CLOCK-RB6"
 		(at 105.41 81.28 0)
-		(fields_autoplaced yes)
 		(effects
 			(font
@@
 	(label "DATA-RB7"
 		(at 229.87 54.61 0)
-		(fields_autoplaced yes)
 		(effects
 			(font
@@
 	(label "CLOCK-RB6"
 		(at 104.14 38.1 0)
-		(fields_autoplaced yes)
 		(effects
 			(font
@@
 	(label "CLOCK-RB6"
 		(at 229.87 57.15 0)
-		(fields_autoplaced yes)
 		(effects
 			(font
@@
 	(label "VCC_PIC"
 		(at 175.26 127 0)
-		(fields_autoplaced yes)
 		(effects
 			(font
@@
 	(label "CLOCK-RB6"
 		(at 229.87 104.14 0)
-		(fields_autoplaced yes)
 		(effects
 			(font
@@
 	(label "VPP-MCLR"
 		(at 179.07 101.6 0)
-		(fields_autoplaced yes)
 		(effects
 			(font
@@
 	(label "VCC_PIC"
 		(at 50.8 63.5 0)
-		(fields_autoplaced yes)
 		(effects
 			(font
@@
 	(label "VCC_PIC"
 		(at 76.2 157.48 0)
-		(fields_autoplaced yes)
 		(effects
 			(font
@@
 	(label "VCC_PIC"
 		(at 232.41 74.93 0)
-		(fields_autoplaced yes)
 		(effects
 			(font
@@
 	(label "VCC_PIC"
 		(at 232.41 121.92 0)
-		(fields_autoplaced yes)
 		(effects
 			(font
@@
 	(label "VPP-MCLR"
 		(at 74.93 154.94 0)
-		(fields_autoplaced yes)
 		(effects
 			(font
@@
 	(label "DATA-RB7"
 		(at 106.68 127 0)
-		(fields_autoplaced yes)
 		(effects
 			(font
@@
 	(label "CLOCK-RB6"
 		(at 106.68 130.81 0)
-		(fields_autoplaced yes)
 		(effects
 			(font
@@
 	(label "VPP-MCLR"
 		(at 179.07 54.61 0)
-		(fields_autoplaced yes)
 		(effects
 			(font
@@
 	(label "DATA-RB7"
 		(at 105.41 71.12 0)
-		(fields_autoplaced yes)
 		(effects
 			(font
@@
 	(label "VPP-MCLR"
 		(at 48.26 88.9 0)
-		(fields_autoplaced yes)
 		(effects
 			(font
@@
 	(label "DATA-RB7"
 		(at 104.14 40.64 0)
-		(fields_autoplaced yes)
 		(effects
 			(font
@@
 	(label "VPP-MCLR"
 		(at 46.99 119.38 0)
-		(fields_autoplaced yes)
 		(effects
 			(font
@@
 	)
 	(symbol
-		(lib_id "flat_hierarchy_schlib:PIC12C508A")
+		(lib_id "flat_hierarchy:PIC12C508A")
 		(at 83.82 76.2 0)
 		(unit 1)
@@
 	)
 	(symbol
-		(lib_id "flat_hierarchy_schlib:PIC16F54")
+		(lib_id "flat_hierarchy:PIC16F54")
 		(at 83.82 123.19 0)
 		(unit 1)
@@
 	)
 	(symbol
-		(lib_id "flat_hierarchy_schlib:GND")
+		(lib_id "flat_hierarchy:GND")
 		(at 101.6 63.5 90)
 		(unit 1)
@@
 	)
 	(symbol
-		(lib_id "flat_hierarchy_schlib:GND")
+		(lib_id "flat_hierarchy:GND")
 		(at 58.42 124.46 0)
 		(unit 1)
@@
 	)
 	(symbol
-		(lib_id "flat_hierarchy_schlib:GND")
+		(lib_id "flat_hierarchy:GND")
 		(at 195.58 129.54 270)
 		(unit 1)
@@
 	)
 	(symbol
-		(lib_id "flat_hierarchy_schlib:24C16")
+		(lib_id "flat_hierarchy:24C16")
 		(at 82.55 35.56 0)
 		(unit 1)
@@
 	)
 	(symbol
-		(lib_id "flat_hierarchy_schlib:GND")
+		(lib_id "flat_hierarchy:GND")
 		(at 59.69 36.83 0)
 		(unit 1)
@@
 	)
 	(symbol
-		(lib_id "flat_hierarchy_schlib:SUPP40")
+		(lib_id "flat_hierarchy:SUPP40")
 		(at 210.82 125.73 0)
 		(unit 1)
@@
 	)
 	(symbol
-		(lib_id "flat_hierarchy_schlib:GND")
+		(lib_id "flat_hierarchy:GND")
 		(at 226.06 124.46 90)
 		(unit 1)
@@
 	)
 	(symbol
-		(lib_id "flat_hierarchy_schlib:C")
+		(lib_id "flat_hierarchy:C")
 		(at 69.85 171.45 0)
 		(unit 1)
@@
 	)
 	(symbol
-		(lib_id "flat_hierarchy_schlib:VCC")
+		(lib_id "flat_hierarchy:VCC")
 		(at 69.85 167.64 0)
 		(unit 1)
@@
 	)
 	(symbol
-		(lib_id "flat_hierarchy_schlib:GND")
+		(lib_id "flat_hierarchy:GND")
 		(at 69.85 176.53 0)
 		(unit 1)
@@
 	)
 	(symbol
-		(lib_id "flat_hierarchy_schlib:C")
+		(lib_id "flat_hierarchy:C")
 		(at 41.91 171.45 0)
 		(unit 1)
@@
 	)
 	(symbol
-		(lib_id "flat_hierarchy_schlib:GND")
+		(lib_id "flat_hierarchy:GND")
 		(at 41.91 176.53 0)
 		(unit 1)
@@
 	)
 	(symbol
-		(lib_id "flat_hierarchy_schlib:SUPP28")
+		(lib_id "flat_hierarchy:SUPP28")
 		(at 210.82 71.12 0)
 		(unit 1)
@@
 	)
 	(symbol
-		(lib_id "flat_hierarchy_schlib:GND")
+		(lib_id "flat_hierarchy:GND")
 		(at 195.58 72.39 270)
 		(unit 1)
@@
 	)
 	(symbol
-		(lib_id "flat_hierarchy_schlib:GND")
+		(lib_id "flat_hierarchy:GND")
 		(at 226.06 77.47 90)
 		(unit 1)
@@
 	)
 	(symbol
-		(lib_id "flat_hierarchy_schlib:GND")
+		(lib_id "flat_hierarchy:GND")
 		(at 195.58 119.38 270)
 		(unit 1)
@@
 	)
 	(symbol
-		(lib_id "flat_hierarchy_schlib:C")
+		(lib_id "flat_hierarchy:C")
 		(at 55.88 171.45 0)
 		(unit 1)
@@
 	)
 	(symbol
-		(lib_id "flat_hierarchy_schlib:GND")
+		(lib_id "flat_hierarchy:GND")
 		(at 55.88 176.53 0)
 		(unit 1)
@@
 	)
 	(symbol
-		(lib_id "flat_hierarchy_schlib:VCC")
+		(lib_id "flat_hierarchy:VCC")
 		(at 82.55 22.86 0)
 		(unit 1)
@@
 	)
 	(symbol
-		(lib_id "flat_hierarchy_schlib:GND")
+		(lib_id "flat_hierarchy:GND")
 		(at 82.55 48.26 0)
 		(unit 1)
