File: demos/kit-dev-coldfire-xilinx_5213/kit-dev-coldfire-xilinx_5213.kicad_sch (KiCad schematic)
At the start: 66 parts, among them Q101 3906, U101 74AHC1G14, U102 MCF5213-LQFP100, Y101 8MHz

Commit message: feat: update kicad to 9.0.0+dfsg-1
Signed-off-by: lhdjply <lhdjply@126.com>
Parts:
- ABRT_SW101, RST_SW101: symbol kit-coldfire_schlib:SW_PUSH -> kit-dev-coldfire-xilinx_5213:SW_PUSH
- ALLPST101, CLKOUT101, GND101, TA-101: symbol kit-coldfire_schlib:CONN_1 -> kit-dev-coldfire-xilinx_5213:CONN_1
- BDM_PORT101: symbol kit-coldfire_schlib:CONN_13X2 -> kit-dev-coldfire-xilinx_5213:CONN_13X2
- C101, C102, C103, C104, C105, C106, C107, C109, C110, C111, C112, C113, C114, C115, C116, C117, C118: symbol kit-coldfire_schlib:C -> kit-dev-coldfire-xilinx_5213:C
- C108, C119: symbol kit-coldfire_schlib:CP -> kit-dev-coldfire-xilinx_5213:CP
- CT101, VDDA101: symbol kit-coldfire_schlib:JUMPER -> kit-dev-coldfire-xilinx_5213:JUMPER
- D101, D102: symbol kit-coldfire_schlib:DIODE -> kit-dev-coldfire-xilinx_5213:DIODE
- FB101, L101, L102: symbol kit-coldfire_schlib:INDUCTOR -> kit-dev-coldfire-xilinx_5213:INDUCTOR
- JP101: symbol kit-coldfire_schlib:JUMPER_TRIPLE -> kit-dev-coldfire-xilinx_5213:JUMPER_TRIPLE
- LEDABRT101, LED_RST101: symbol kit-coldfire_schlib:LED -> kit-dev-coldfire-xilinx_5213:LED
- LV101: symbol kit-coldfire_schlib:MC34064P -> kit-dev-coldfire-xilinx_5213:MC34064P
- Q101: symbol kit-coldfire_schlib:PNP -> kit-dev-coldfire-xilinx_5213:PNP
- R101, R102, R103, R104, R105, R106, R107, R108, R109, R110, R111, R112, R113, R114, R115, R116, R117, R118, R119, R120, R121, R122, R123, R124, R125: symbol kit-coldfire_schlib:R -> kit-dev-coldfire-xilinx_5213:R
- U101: symbol kit-coldfire_schlib:74AHC1G14 -> kit-dev-coldfire-xilinx_5213:74AHC1G14
- U102: symbol kit-coldfire_schlib:MCF5213-LQFP100 -> kit-dev-coldfire-xilinx_5213:MCF5213-LQFP100
- Y101: symbol kit-coldfire_schlib:CRYSTAL -> kit-dev-coldfire-xilinx_5213:CRYSTAL
