File: demos/pic_programmer/pic_sockets.kicad_sch (KiCad schematic)
At the start: 7 parts, among them P2 SUPP28, P3 SUPP40, U1 24Cxx, U5 PIC_18_PINS, U6 PIC_8_PINS

Commit message: feat: update kicad to 9.0.0+dfsg-1
Signed-off-by: lhdjply <lhdjply@126.com>
Parts:
- C6, C7: symbol pic_programmer_schlib:C -> pic_programmer:C
- P2: symbol pic_programmer_schlib:SUPP28 -> pic_programmer:SUPP28
- P3: symbol pic_programmer_schlib:SUPP40 -> pic_programmer:SUPP40
- U1: symbol pic_programmer_schlib:24C16 -> pic_programmer:24C16
- U5: symbol pic_programmer_schlib:PIC16F54 -> pic_programmer:PIC16F54
- U6: symbol pic_programmer_schlib:PIC12C508A -> pic_programmer:PIC12C508A
Changed lines of the file:
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@@
 (kicad_sch
-	(version 20231120)
+	(version 20250114)
 	(generator "eeschema")
-	(generator_version "8.0")
+	(generator_version "9.0")
 	(paper "A4")
 	(title_block
@@
 	(label "DATA-RB7"
 		(at 237.49 48.26 0)
-		(fields_autoplaced yes)
 		(effects
 			(font
@@
 	(label "CLOCK-RB6"
 		(at 118.11 124.46 0)
-		(fields_autoplaced yes)
 		(effects
 			(font
@@
 	(label "CLOCK-RB6"
 		(at 237.49 101.6 0)
-		(fields_autoplaced yes)
 		(effects
 			(font
@@
 	(label "VCC_PIC"
 		(at 93.98 20.32 0)
-		(fields_autoplaced yes)
 		(effects
 			(font
@@
 	(label "VCC_PIC"
 		(at 240.03 119.38 0)
-		(fields_autoplaced yes)
 		(effects
 			(font
@@
 	(label "VCC_PIC"
 		(at 182.88 124.46 0)
-		(fields_autoplaced yes)
 		(effects
 			(font
@@
 	(label "VCC_PIC"
 		(at 120.65 116.84 0)
-		(fields_autoplaced yes)
 		(effects
 			(font
@@
 	(label "VCC_PIC"
 		(at 69.85 165.1 0)
-		(fields_autoplaced yes)
 		(effects
 			(font
@@
 	(label "DATA-RB7"
 		(at 115.57 38.1 0)
-		(fields_autoplaced yes)
 		(effects
 			(font
@@
 	(label "DATA-RB7"
 		(at 118.11 120.65 0)
-		(fields_autoplaced yes)
 		(effects
 			(font
@@
 	(label "VPP-MCLR"
 		(at 58.42 113.03 0)
-		(fields_autoplaced yes)
 		(effects
 			(font
@@
 	(label "VPP-MCLR"
 		(at 59.69 86.36 0)
-		(fields_autoplaced yes)
 		(effects
 			(font
@@
 	(label "VPP-MCLR"
 		(at 186.69 99.06 0)
-		(fields_autoplaced yes)
 		(effects
 			(font
@@
 	(label "VPP-MCLR"
 		(at 186.69 48.26 0)
-		(fields_autoplaced yes)
 		(effects
 			(font
@@
 	(label "VCC_PIC"
 		(at 62.23 60.96 0)
-		(fields_autoplaced yes)
 		(effects
 			(font
@@
 	(label "VCC_PIC"
 		(at 240.03 68.58 0)
-		(fields_autoplaced yes)
 		(effects
 			(font
@@
 	(label "DATA-RB7"
 		(at 237.49 99.06 0)
-		(fields_autoplaced yes)
 		(effects
 			(font
@@
 	(label "CLOCK-RB6"
 		(at 116.84 78.74 0)
-		(fields_autoplaced yes)
 		(effects
 			(font
@@
 	(label "DATA-RB7"
 		(at 116.84 68.58 0)
-		(fields_autoplaced yes)
 		(effects
 			(font
@@
 	(label "CLOCK-RB6"
 		(at 237.49 50.8 0)
-		(fields_autoplaced yes)
 		(effects
 			(font
@@
 	(label "CLOCK-RB6"
 		(at 115.57 35.56 0)
-		(fields_autoplaced yes)
 		(effects
 			(font
@@
 		(shape input)
 		(at 48.26 50.8 180)
-		(fields_autoplaced yes)
 		(effects
 			(font
@@
 		(shape input)
 		(at 48.26 53.34 180)
-		(fields_autoplaced yes)
 		(effects
 			(font
@@
 		(shape input)
 		(at 48.26 160.02 180)
-		(fields_autoplaced yes)
 		(effects
 			(font
@@
 		(shape input)
 		(at 48.26 157.48 180)
-		(fields_autoplaced yes)
 		(effects
 			(font
@@
 	)
 	(symbol
-		(lib_id "pic_programmer_schlib:PIC12C508A")
+		(lib_id "pic_programmer:PIC12C508A")
 		(at 95.25 73.66 0)
 		(unit 1)
@@
 	)
 	(symbol
-		(lib_id "pic_programmer_schlib:PIC16F54")
+		(lib_id "pic_programmer:PIC16F54")
 		(at 95.25 116.84 0)
 		(unit 1)
@@
 	)
 	(symbol
-		(lib_id "pic_programmer_schlib:GND")
+		(lib_id "pic_programmer:GND")
 		(at 113.03 60.96 90)
 		(unit 1)
@@
 	)
 	(symbol
-		(lib_id "pic_programmer_schlib:GND")
+		(lib_id "pic_programmer:GND")
 		(at 69.85 118.11 0)
 		(unit 1)
@@
 	)
 	(symbol
-		(lib_id "pic_programmer_schlib:GND")
+		(lib_id "pic_programmer:GND")
 		(at 203.2 127 270)
 		(unit 1)
@@
 	)
 	(symbol
-		(lib_id "pic_programmer_schlib:24C16")
+		(lib_id "pic_programmer:24C16")
 		(at 93.98 33.02 0)
 		(unit 1)
@@
 	)
 	(symbol
-		(lib_id "pic_programmer_schlib:GND")
+		(lib_id "pic_programmer:GND")
 		(at 71.12 34.29 0)
 		(unit 1)
@@
 	)
 	(symbol
-		(lib_id "pic_programmer_schlib:SUPP40")
+		(lib_id "pic_programmer:SUPP40")
 		(at 218.44 123.19 0)
 		(unit 1)
@@
 	)
 	(symbol
-		(lib_id "pic_programmer_schlib:GND")
+		(lib_id "pic_programmer:GND")
 		(at 233.68 121.92 90)
 		(unit 1)
@@
 	)
 	(symbol
-		(lib_id "pic_programmer_schlib:C")
+		(lib_id "pic_programmer:C")
 		(at 60.96 171.45 0)
 		(unit 1)
@@
 	)
 	(symbol
-		(lib_id "pic_programmer_schlib:GND")
+		(lib_id "pic_programmer:GND")
 		(at 60.96 176.53 0)
 		(unit 1)
@@
 	)
 	(symbol
-		(lib_id "pic_programmer_schlib:C")
+		(lib_id "pic_programmer:C")
 		(at 83.82 171.45 0)
 		(unit 1)
@@
 	)
 	(symbol
-		(lib_id "pic_programmer_schlib:GND")
+		(lib_id "pic_programmer:GND")
 		(at 83.82 176.53 0)
 		(unit 1)
@@
 	)
 	(symbol
-		(lib_id "pic_programmer_schlib:SUPP28")
+		(lib_id "pic_programmer:SUPP28")
 		(at 218.44 64.77 0)
 		(unit 1)
@@
 	)
 	(symbol
-		(lib_id "pic_programmer_schlib:GND")
+		(lib_id "pic_programmer:GND")
 		(at 203.2 66.04 270)
 		(unit 1)
@@
 	)
 	(symbol
-		(lib_id "pic_programmer_schlib:GND")
+		(lib_id "pic_programmer:GND")
 		(at 233.68 71.12 90)
 		(unit 1)
@@
 	)
 	(symbol
-		(lib_id "pic_programmer_schlib:GND")
+		(lib_id "pic_programmer:GND")
 		(at 203.2 116.84 270)
 		(unit 1)
@@
 	)
 	(symbol
-		(lib_id "pic_programmer_schlib:GND")
+		(lib_id "pic_programmer:GND")
 		(at 93.98 46.99 0)
 		(unit 1)
@@
 	)
 	(symbol
-		(lib_id "pic_programmer_schlib:PWR_FLAG")
+		(lib_id "pic_programmer:PWR_FLAG")
 		(at 83.82 165.1 270)
 		(unit 1)
