File: demos/simulation/class-d/Class-D.kicad_sch (KiCad schematic)
At the start: 39 parts, among them Q1 NPN, Q2 NMOS, Q3 NPN, Q4 PNP, Q5 PNP, Q6 NMOS, U1 AudioDriver1

Commit message: feat: update kicad to 9.0.0+dfsg-1
Signed-off-by: lhdjply <lhdjply@126.com>
Changed lines of the file:
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@@
 (kicad_sch
-	(version 20231120)
+	(version 20241209)
 	(generator "eeschema")
-	(generator_version "8.0")
+	(generator_version "9.0")
 	(paper "A4")
 	(title_block
@@
 		(comment 4 "Circuit idea:")
 	)
+	(text ".options chgtol=1e-11 abstol=1u \n.probe p(R15)\n.control\nset controlswait\nrusage time\n.endc\n"
+		(exclude_from_sim no)
+		(at 95.885 116.84 0)
+		(effects
+			(font
+				(size 1.27 1.27)
+			)
+			(justify left)
+		)
+	)
+	(text "Analog input\nPulse Width Modulator\nComplementary push-pull clock\nDead time to avoid shoot-through current\nHigh side voltage shift"
+		(exclude_from_sim no)
+		(at 79.375 46.99 0)
+		(effects
+			(font
+				(size 1.27 1.27)
+			)
+			(justify left)
+		)
+	)
 	(junction
 		(at 182.88 86.36)
@@
 		)
 	)
-	(text ".options chgtol=1e-11 abstol=1u \n.probe p(R15)\n.control\nset controlswait\nrusage time\n.endc\n"
-		(exclude_from_sim no)
-		(at 95.885 116.84 0)
-		(effects
-			(font
-				(size 1.27 1.27)
-			)
-			(justify left)
-		)
-	)
-	(text "Analog input\nPulse Width Modulator\nComplementary push-pull clock\nDead time to avoid shoot-through current\nHigh side voltage shift"
-		(exclude_from_sim no)
-		(at 79.375 46.99 0)
-		(effects
-			(font
-				(size 1.27 1.27)
-			)
-			(justify left)
-		)
-	)
 	(label "B-"
 		(at 204.47 138.43 0)
-		(fields_autoplaced yes)
 		(effects
 			(font
@@
 	(label "B+"
 		(at 215.9 36.83 0)
-		(fields_autoplaced yes)
 		(effects
 			(font
@@
 	(label "Vs"
 		(at 248.92 132.08 0)
-		(fields_autoplaced yes)
 		(effects
 			(font
@@
 	(label "out"
 		(at 276.86 66.04 0)
-		(fields_autoplaced yes)
 		(effects
 			(font
@@
 	(label "B+"
 		(at 204.47 110.49 0)
-		(fields_autoplaced yes)
 		(effects
 			(font
@@
 	(label "Ain"
 		(at 156.21 114.3 0)
-		(fields_autoplaced yes)
 		(effects
 			(font
@@
 	(label "Vcc"
 		(at 130.81 73.66 0)
-		(fields_autoplaced yes)
 		(effects
 			(font
@@
 	(label "Vb"
 		(at 248.92 116.84 0)
-		(fields_autoplaced yes)
 		(effects
 			(font
@@
 	(label "Fb1"
 		(at 222.25 27.94 0)
-		(fields_autoplaced yes)
 		(effects
 			(font
@@
 	(label "Vcc"
 		(at 232.41 116.84 0)
-		(fields_autoplaced yes)
 		(effects
 			(font
@@
 	(label "HO"
 		(at 130.81 48.26 0)
-		(fields_autoplaced yes)
 		(effects
 			(font
@@
 	(label "B-"
 		(at 217.17 104.14 0)
-		(fields_autoplaced yes)
 		(effects
 			(font
@@
 	(label "LO"
 		(at 130.81 86.36 0)
-		(fields_autoplaced yes)
 		(effects
 			(font
@@
 	(label "out"
 		(at 267.97 118.11 0)
-		(fields_autoplaced yes)
 		(effects
 			(font
@@
 	(label "Vb"
 		(at 130.81 35.56 0)
-		(fields_autoplaced yes)
 		(effects
 			(font
@@
 	(label "B-"
 		(at 132.08 104.14 0)
-		(fields_autoplaced yes)
 		(effects
 			(font
@@
 	(label "Ain"
 		(at 92.71 68.58 0)
-		(fields_autoplaced yes)
 		(effects
 			(font
@@
 	(label "B-"
 		(at 232.41 132.08 0)
-		(fields_autoplaced yes)
 		(effects
 			(font
@@
 	(label "Fb2"
 		(at 251.46 27.94 0)
-		(fields_autoplaced yes)
 		(effects
 			(font
@@
 	(label "Vs"
 		(at 130.81 66.04 0)
-		(fields_autoplaced yes)
 		(effects
 			(font
@@
 		)
 	)
+	(embedded_fonts no)
 )
