File: demos/sonde xilinx/sonde xilinx.kicad_pcb (KiCad board)
At the start: 2 copper layers, 80.4 x 43.2 mm, 25 parts, among them J1 DB25MALE, J2 DB9MALE, P1 CONN_6, U1 74LS125, U2 74LS125

Commit message: feat: update kicad to 9.0.0+dfsg-1
Signed-off-by: lhdjply <lhdjply@126.com>
Parts:
- C1: footprint Capacitor_THT:C_Axial_L5.1mm_D3.1mm_P12.50mm_Horizontal -> sonde-xilinx:C_Axial_L5.1mm_D3.1mm_P12.50mm_Horizontal
- C2, C3, C4, C5: footprint Capacitor_THT:C_Disc_D5.1mm_W3.2mm_P5.00mm -> sonde-xilinx:C_Disc_D5.1mm_W3.2mm_P5.00mm
- D1, D2: footprint Diode_THT:D_A-405_P7.62mm_Horizontal -> sonde-xilinx:D_A-405_P7.62mm_Horizontal
- J1: footprint Connector_Dsub:DSUB-25_Male_EdgeMount_P2.77mm -> sonde-xilinx:DSUB-25_Male_EdgeMount_P2.77mm
- J2: footprint Connector_Dsub:DSUB-9_Male_EdgeMount_P2.77mm -> sonde-xilinx:DSUB-9_Male_EdgeMount_P2.77mm
- P1: footprint Connector_PinHeader_2.54mm:PinHeader_1x06_P2.54mm_Vertical -> sonde-xilinx:PinHeader_1x06_P2.54mm_Vertical
- R1, R10, R11, R12, R13, R14, R2, R4, R5, R6, R7, R8, R9: footprint Resistor_THT:R_Axial_DIN0207_L6.3mm_D2.5mm_P10.16mm_Horizontal -> sonde-xilinx:R_Axial_DIN0207_L6.3mm_D2.5mm_P10.16mm_Horizontal
- U1, U2: footprint Package_DIP:DIP-14_W7.62mm_LongPads -> sonde-xilinx:DIP-14_W7.62mm_LongPads
