File: demos/video/pal-ntsc.kicad_sch (KiCad schematic)
At the start: 36 parts, among them U10 BT812, X2 30MHz

Commit message: feat: update kicad to 9.0.0+dfsg-1
Signed-off-by: lhdjply <lhdjply@126.com>
Changed lines of the file:
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@@
 (kicad_sch
-	(version 20231120)
+	(version 20250114)
 	(generator "eeschema")
-	(generator_version "8.0")
+	(generator_version "9.0")
 	(paper "A3")
 	(title_block
@@
 	(label "VAF"
 		(at 257.81 60.96 180)
-		(fields_autoplaced yes)
 		(effects
 			(font
@@
 	(label "PC_D5"
 		(at 138.43 198.12 0)
-		(fields_autoplaced yes)
 		(effects
 			(font
@@
 	(label "TVG1"
 		(at 257.81 106.68 0)
-		(fields_autoplaced yes)
 		(effects
 			(font
@@
 	(label "TVR1"
 		(at 257.81 83.82 0)
-		(fields_autoplaced yes)
 		(effects
 			(font
@@
 	(label "TVB6"
 		(at 257.81 142.24 0)
-		(fields_autoplaced yes)
 		(effects
 			(font
@@
 	(label "TVB5"
 		(at 257.81 139.7 0)
-		(fields_autoplaced yes)
 		(effects
 			(font
@@
 	(label "TVB3"
 		(at 257.81 134.62 0)
-		(fields_autoplaced yes)
 		(effects
 			(font
@@
 	(label "TVR7"
 		(at 257.81 99.06 0)
-		(fields_autoplaced yes)
 		(effects
 			(font
@@
 	(label "TVR3"
 		(at 257.81 88.9 0)
-		(fields_autoplaced yes)
 		(effects
 			(font
@@
 	(label "TVG4"
 		(at 257.81 114.3 0)
-		(fields_autoplaced yes)
 		(effects
 			(font
@@
 	(label "TVB0"
 		(at 257.81 127 0)
-		(fields_autoplaced yes)
 		(effects
 			(font
@@
 	(label "Y_SYNC"
 		(at 257.81 154.94 0)
-		(fields_autoplaced yes)
 		(effects
 			(font
@@
 	(label "TVG6"
 		(at 257.81 119.38 0)
-		(fields_autoplaced yes)
 		(effects
 			(font
@@
 	(label "VAF"
 		(at 288.29 45.72 180)
-		(fields_autoplaced yes)
 		(effects
 			(font
@@
 	(label "TVR0"
 		(at 257.81 81.28 0)
-		(fields_autoplaced yes)
 		(effects
 			(font
@@
 	(label "TVB4"
 		(at 257.81 137.16 0)
-		(fields_autoplaced yes)
 		(effects
 			(font
@@
 	(label "PC_D2"
 		(at 138.43 190.5 0)
-		(fields_autoplaced yes)
 		(effects
 			(font
@@
 	(label "TVR6"
 		(at 257.81 96.52 0)
-		(fields_autoplaced yes)
 		(effects
 			(font
@@
 	(label "TVG7"
 		(at 257.81 121.92 0)
-		(fields_autoplaced yes)
 		(effects
 			(font
@@
 	(label "TVG0"
 		(at 257.81 104.14 0)
-		(fields_autoplaced yes)
 		(effects
 			(font
@@
 	(label "TVR2"
 		(at 257.81 86.36 0)
-		(fields_autoplaced yes)
 		(effects
 			(font
@@
 	(label "PC_A1"
 		(at 138.43 210.82 0)
-		(fields_autoplaced yes)
 		(effects
 			(font
@@
 	(label "TVR5"
 		(at 257.81 93.98 0)
-		(fields_autoplaced yes)
 		(effects
 			(font
@@
 	(label "VAF"
 		(at 293.37 76.2 0)
-		(fields_autoplaced yes)
 		(effects
 			(font
@@
 	(label "VAF"
 		(at 118.11 180.34 0)
-		(fields_autoplaced yes)
 		(effects
 			(font
@@
 	(label "PC_A0"
 		(at 138.43 208.28 0)
-		(fields_autoplaced yes)
 		(effects
 			(font
@@
 	(label "TVB7"
 		(at 257.81 144.78 0)
-		(fields_autoplaced yes)
 		(effects
 			(font
@@
 	(label "Y-VIDEO"
 		(at 128.27 116.84 0)
-		(fields_autoplaced yes)
 		(effects
 			(font
@@
 	(label "C-VIDEO"
 		(at 128.27 119.38 0)
-		(fields_autoplaced yes)
 		(effects
 			(font
@@
 	(label "TVB2"
 		(at 257.81 132.08 0)
-		(fields_autoplaced yes)
 		(effects
 			(font
@@
 	(label "TVR4"
 		(at 257.81 91.44 0)
-		(fields_autoplaced yes)
 		(effects
 			(font
@@
 	(label "PC_D0"
 		(at 138.43 185.42 0)
-		(fields_autoplaced yes)
 		(effects
 			(font
@@
 	(label "TVG5"
 		(at 257.81 116.84 0)
-		(fields_autoplaced yes)
 		(effects
 			(font
@@
 	(label "TVG2"
 		(at 257.81 109.22 0)
-		(fields_autoplaced yes)
 		(effects
 			(font
@@
 	(label "TVG3"
 		(at 257.81 111.76 0)
-		(fields_autoplaced yes)
 		(effects
 			(font
@@
 	(label "PC_D3"
 		(at 138.43 193.04 0)
-		(fields_autoplaced yes)
 		(effects
 			(font
@@
 	(label "PC_D6"
 		(at 138.43 200.66 0)
-		(fields_autoplaced yes)
 		(effects
 			(font
@@
 	(label "PC_D4"
 		(at 138.43 195.58 0)
-		(fields_autoplaced yes)
 		(effects
 			(font
@@
 	(label "PC_D7"
 		(at 138.43 203.2 0)
-		(fields_autoplaced yes)
 		(effects
 			(font
@@
 	(label "PC_D1"
 		(at 138.43 187.96 0)
-		(fields_autoplaced yes)
 		(effects
 			(font
@@
 	(label "TVB1"
 		(at 257.81 129.54 0)
-		(fields_autoplaced yes)
 		(effects
 			(font
@@
 	(label "Y_SYNC"
 		(at 52.07 165.1 0)
-		(fields_autoplaced yes)
 		(effects
 			(font
@@
 		(shape bidirectional)
 		(at 274.32 124.46 0)
-		(fields_autoplaced yes)
 		(effects
 			(font
@@
 		(shape input)
 		(at 151.13 215.9 180)
-		(fields_autoplaced yes)
 		(effects
 			(font
@@
 		(shape input)
 		(at 151.13 218.44 180)
-		(fields_autoplaced yes)
 		(effects
 			(font
@@
 		(shape input)
 		(at 147.32 96.52 180)
-		(fields_autoplaced yes)
 		(effects
 			(font
@@
 		(shape input)
 		(at 64.77 40.64 180)
-		(fields_autoplaced yes)
 		(effects
 			(font
@@
 		(shape output)
 		(at 257.81 193.04 0)
-		(fields_autoplaced yes)
 		(effects
 			(font
@@
 		(shape bidirectional)
 		(at 274.32 78.74 0)
-		(fields_autoplaced yes)
 		(effects
 			(font
@@
 		(shape bidirectional)
 		(at 64.77 38.1 180)
-		(fields_autoplaced yes)
 		(effects
 			(font
@@
 		(shape output)
 		(at 257.81 215.9 0)
-		(fields_autoplaced yes)
 		(effects
 			(font
@@
 		(shape output)
 		(at 257.81 190.5 0)
-		(fields_autoplaced yes)
 		(effects
 			(font
@@
 		(shape bidirectional)
 		(at 274.32 101.6 0)
-		(fields_autoplaced yes)
 		(effects
 			(font
@@
 		(shape input)
 		(at 72.39 106.68 180)
-		(fields_autoplaced yes)
 		(effects
 			(font
@@
 		(shape input)
 		(at 151.13 223.52 180)
-		(fields_autoplaced yes)
 		(effects
 			(font
@@
 		(shape input)
 		(at 72.39 129.54 180)
-		(fields_autoplaced yes)
 		(effects
 			(font
